Commit message: Update racecar.xacro

File: velma/src/pathing/racecar.xacro (robot description, xacro)
@@ -67,39 +67,5 @@
     </visual>
   </link>
-<!--  <joint name="base_to_front_left_hinge" type="fixed">
-    <parent link="base_link"/>
-    <child link="front_left_hinge"/>
-    <origin xyz="${wheelbase} ${(wheel_length+width)/2} ${wheel_radius}"/>
-  </joint> -->
-  <joint name="base_to_front_left_wheel" type="fixed">
-    <parent link="base_link"/>
-    <child link="front_left_wheel"/>
-    <origin xyz="${wheelbase} ${(wheel_length+width)/2} ${wheel_radius}"/>
-  </joint>
-  <!--<link name="front_left_hinge"/>
-  <joint name="front_left_hinge_to_wheel" type="continuous">
-    <parent link="front_left_hinge"/>
-    <child link="front_left_wheel"/>
-  </joint> -->
-  <link name="front_left_wheel">
-    <visual>
-      <geometry>
-        <cylinder radius="${wheel_radius}" length="${wheel_length}"/>
-      </geometry>
-      <material name="black"/>
-      <origin rpy="${pi/2} 0 0"/>
-    </visual>
-  </link>
-  <!--<joint name="base_to_front_right_hinge" type="fixed">
-    <parent link="base_link"/>
-    <child link="front_right_hinge"/>
-    <origin xyz="${wheelbase} ${-(wheel_length+width)/2} ${wheel_radius}"/>
-  </joint>-->
-  <!--<link name="front_right_hinge"/>
-  <joint name="front_right_hinge_to_wheel" type="continuous">
-    <parent link="front_right_hinge"/>
-    <child link="front_right_wheel"/>
-  </joint> -->
-    <joint name="base_to_front_right_wheel" type="fixed">
+  <joint name="base_to_front_right_wheel" type="fixed">
     <parent link="base_link"/>
     <child link="front_right_wheel"/>
@@ -115,3 +81,51 @@
     </visual>
   </link>
+  <joint name="base_to_front_left_wheel" type="fixed">
+    <parent link="base_link"/>
+    <child link="front_left_wheel"/>
+    <origin xyz="${wheelbase} ${(wheel_length+width)/2} ${wheel_radius}"/>
+  </joint>
+  <link name="front_left_wheel">
+    <visual>
+      <geometry>
+        <cylinder radius="${wheel_radius}" length="${wheel_length}"/>
+      </geometry>
+      <material name="black"/>
+      <origin rpy="${pi/2} 0 0"/>
+    </visual>
+  </link>
+  <joint name="base_to_front_right_wheel" type="fixed">
+    <parent link="base_link"/>
+    <child link="front_right_wheel"/>
+    <origin xyz="${wheelbase} ${-(wheel_length+width)/2} ${wheel_radius}"/>
+  </joint>
+  <link name="front_right_wheel">
+    <visual>
+      <geometry>
+        <cylinder radius="${wheel_radius}" length="${wheel_length}"/>
+      </geometry>
+      <material name="black"/>
+      <origin rpy="${pi/2} 0 0"/>
+    </visual>
+  </link>
+<!--  <joint name="base_to_front_left_hinge" type="fixed">
+    <parent link="base_link"/>
+    <child link="front_left_hinge"/>
+    <origin xyz="${wheelbase} ${(wheel_length+width)/2} ${wheel_radius}"/>
+  </joint> -->
+  <!--<link name="front_left_hinge"/>
+  <joint name="front_left_hinge_to_wheel" type="continuous">
+    <parent link="front_left_hinge"/>
+    <child link="front_left_wheel"/>
+  </joint> -->
+  <!--<joint name="base_to_front_right_hinge" type="fixed">
+    <parent link="base_link"/>
+    <child link="front_right_hinge"/>
+    <origin xyz="${wheelbase} ${-(wheel_length+width)/2} ${wheel_radius}"/>
+  </joint>-->
+  <!--<link name="front_right_hinge"/>
+  <joint name="front_right_hinge_to_wheel" type="continuous">
+    <parent link="front_right_hinge"/>
+    <child link="front_right_wheel"/>
+  </joint> -->
 </robot>

Commit message: Update racecar.xacro

File: velma/src/pathing/racecar.xacro (robot description, xacro)
@@ -95,18 +95,4 @@
     </visual>
   </link>
-  <joint name="base_to_front_right_wheel" type="fixed">
-    <parent link="base_link"/>
-    <child link="front_right_wheel"/>
-    <origin xyz="${wheelbase} ${-(wheel_length+width)/2} ${wheel_radius}"/>
-  </joint>
-  <link name="front_right_wheel">
-    <visual>
-      <geometry>
-        <cylinder radius="${wheel_radius}" length="${wheel_length}"/>
-      </geometry>
-      <material name="black"/>
-      <origin rpy="${pi/2} 0 0"/>
-    </visual>
-  </link>
 <!--  <joint name="base_to_front_left_hinge" type="fixed">
     <parent link="base_link"/>

Commit message: update

File: velma/src/pathing/racecar.xacro (robot description, xacro)
@@ -17,5 +17,5 @@
     <color rgba="0.3 0.57 1. 1."/>
   </material>
-  <link name="base_link">
+  <link name="base_footprint">
     <visual>
       <origin xyz="${wheelbase/2} 0 ${ground_offset+height/2}"/>
@@ -27,5 +27,5 @@
   </link>
   <joint name="base_to_laser_model" type="fixed">
-    <parent link="base_link"/>
+    <parent link="base_footprint"/>
     <child link="laser_model"/>
     <origin xyz="${laser_distance_from_base_link} 0 ${ground_offset+height+(laser_height/2)}"/>
@@ -40,5 +40,5 @@
   </link>
   <joint name="base_to_back_left_wheel" type="fixed">
-    <parent link="base_link"/>
+    <parent link="base_footprint"/>
     <child link="back_left_wheel"/>
     <origin xyz="0 ${(wheel_length+width)/2} ${wheel_radius}"/>
@@ -54,5 +54,5 @@
   </link>
   <joint name="base_to_back_right_wheel" type="fixed">
-    <parent link="base_link"/>
+    <parent link="base_footprint"/>
     <child link="back_right_wheel"/>
     <origin xyz="0 ${-(wheel_length+width)/2} ${wheel_radius}"/>
@@ -68,5 +68,5 @@
   </link>
   <joint name="base_to_front_right_wheel" type="fixed">
-    <parent link="base_link"/>
+    <parent link="base_footprint"/>
     <child link="front_right_wheel"/>
     <origin xyz="${wheelbase} ${-(wheel_length+width)/2} ${wheel_radius}"/>
@@ -82,5 +82,5 @@
   </link>
   <joint name="base_to_front_left_wheel" type="fixed">
-    <parent link="base_link"/>
+    <parent link="base_footprint"/>
     <child link="front_left_wheel"/>
     <origin xyz="${wheelbase} ${(wheel_length+width)/2} ${wheel_radius}"/>
